File: Schematic/Inertial Sensors.kicad_sch (KiCad schematic)
At the start: 14 parts, among them U6 ICM-45686, U7 ADXL375, U8 LIS2MDL, U9 MS5607-02BA

Commit message: Made board smaller
Parts:
- renumbered C21 to C22, C22 to C23, C23 to C24, C24 to C25, C25 to C26, C26 to C27, C27 to C28, C28 to C29, C29 to C30, C30 to C31
Changed lines of the file:
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@@
 		(title "Icarus Flight Computer")
 		(date "2025-04-30")
-		(rev "1.0")
+		(rev "V1.0")
 		(company "Daedalus Industries")
 		(comment 1 "Onboard flight computer for the Icarus rocket")
 		(comment 2 "Sensors for orientation and velocity estimation")
+		(comment 3 "Designer: Mattia Gregnanin")
 	)
 	(rectangle
@@
 		(on_board yes)
 		(dnp no)
-		(property "Reference" "#PWR062"
+		(property "Reference" "#PWR067"
 			(at 69.85 116.84 0)
 			(effects
@@
 			(project "Icarus Flight Computer"
 				(path "/2a10c6de-1617-4216-ace2-cdde3ce2909e/3d2049bb-024c-4c55-ac2e-c537e2a25c23"
-					(reference "#PWR062")
+					(reference "#PWR067")
 					(unit 1)
 				)
@@
 		(on_board yes)
 		(dnp no)
-		(property "Reference" "#PWR065"
+		(property "Reference" "#PWR070"
 			(at 105.41 127 0)
 			(effects
@@
 			(project "Icarus Flight Computer"
 				(path "/2a10c6de-1617-4216-ace2-cdde3ce2909e/3d2049bb-024c-4c55-ac2e-c537e2a25c23"
-					(reference "#PWR065")
+					(reference "#PWR070")
 					(unit 1)
 				)
@@
 		(on_board yes)
 		(dnp no)
-		(property "Reference" "#PWR054"
+		(property "Reference" "#PWR059"
 			(at 182.88 48.26 0)
 			(effects
@@
 			(project "Icarus Flight Computer"
 				(path "/2a10c6de-1617-4216-ace2-cdde3ce2909e/3d2049bb-024c-4c55-ac2e-c537e2a25c23"
-					(reference "#PWR054")
+					(reference "#PWR059")
 					(unit 1)
 				)
@@
 		(on_board yes)
 		(dnp no)
-		(property "Reference" "#PWR069"
+		(property "Reference" "#PWR074"
 			(at 69.85 149.86 0)
 			(effects
@@
 			(project "Icarus Flight Computer"
 				(path "/2a10c6de-1617-4216-ace2-cdde3ce2909e/3d2049bb-024c-4c55-ac2e-c537e2a25c23"
-					(reference "#PWR069")
+					(reference "#PWR074")
 					(unit 1)
 				)
@@
 		(on_board yes)
 		(dnp no)
-		(property "Reference" "#PWR067"
+		(property "Reference" "#PWR072"
 			(at 105.41 142.24 0)
 			(effects
@@
 			(project "Icarus Flight Computer"
 				(path "/2a10c6de-1617-4216-ace2-cdde3ce2909e/3d2049bb-024c-4c55-ac2e-c537e2a25c23"
-					(reference "#PWR067")
+					(reference "#PWR072")
 					(unit 1)
 				)
@@
 		(dnp no)
 		(fields_autoplaced yes)
-		(property "Reference" "C28"
+		(property "Reference" "C29"
 			(at 120.65 128.2699 0)
 			(effects
@@
 			(project "Icarus Flight Computer"
 				(path "/2a10c6de-1617-4216-ace2-cdde3ce2909e/3d2049bb-024c-4c55-ac2e-c537e2a25c23"
-					(reference "C28")
+					(reference "C29")
 					(unit 1)
 				)
@@
 		(on_board yes)
 		(dnp no)
-		(property "Reference" "#PWR060"
+		(property "Reference" "#PWR065"
 			(at 76.2 81.28 0)
 			(effects
@@
 			(project "Icarus Flight Computer"
 				(path "/2a10c6de-1617-4216-ace2-cdde3ce2909e/3d2049bb-024c-4c55-ac2e-c537e2a25c23"
-					(reference "#PWR060")
+					(reference "#PWR065")
 					(unit 1)
 				)
@@
 		(dnp no)
 		(fields_autoplaced yes)
-		(property "Reference" "C22"
+		(property "Reference" "C23"
 			(at 124.46 58.4199 0)
 			(effects
@@
 			(project "Icarus Flight Computer"
 				(path "/2a10c6de-1617-4216-ace2-cdde3ce2909e/3d2049bb-024c-4c55-ac2e-c537e2a25c23"
-					(reference "C22")
+					(reference "C23")
 					(unit 1)
 				)
@@
 		(on_board yes)
 		(dnp no)
-		(property "Reference" "#PWR066"
+		(property "Reference" "#PWR071"
 			(at 215.9 140.97 0)
 			(effects
@@
 			(project "Icarus Flight Computer"
 				(path "/2a10c6de-1617-4216-ace2-cdde3ce2909e/3d2049bb-024c-4c55-ac2e-c537e2a25c23"
-					(reference "#PWR066")
+					(reference "#PWR071")
 					(unit 1)
 				)
@@
 		(dnp no)
 		(fields_autoplaced yes)
-		(property "Reference" "C26"
+		(property "Reference" "C27"
 			(at 219.71 126.9999 0)
 			(effects
@@
 			(project "Icarus Flight Computer"
 				(path "/2a10c6de-1617-4216-ace2-cdde3ce2909e/3d2049bb-024c-4c55-ac2e-c537e2a25c23"
-					(reference "C26")
+					(reference "C27")
 					(unit 1)
 				)
@@
 		(dnp no)
 		(fields_autoplaced yes)
-		(property "Reference" "C30"
+		(property "Reference" "C31"
 			(at 91.44 135.8899 0)
 			(effects
@@
 			(project ""
 				(path "/2a10c6de-1617-4216-ace2-cdde3ce2909e/3d2049bb-024c-4c55-ac2e-c537e2a25c23"
-					(reference "C30")
+					(reference "C31")
 					(unit 1)
 				)
@@
 		(dnp no)
 		(fields_autoplaced yes)
-		(property "Reference" "C27"
+		(property "Reference" "C28"
 			(at 109.22 128.2699 0)
 			(effects
@@
 			(project "Icarus Flight Computer"
 				(path "/2a10c6de-1617-4216-ace2-cdde3ce2909e/3d2049bb-024c-4c55-ac2e-c537e2a25c23"
-					(reference "C27")
+					(reference "C28")
 					(unit 1)
 				)
@@
 		(on_board yes)
 		(dnp no)
-		(property "Reference" "#PWR058"
+		(property "Reference" "#PWR063"
 			(at 214.63 73.66 0)
 			(effects
@@
 			(project "Icarus Flight Computer"
 				(path "/2a10c6de-1617-4216-ace2-cdde3ce2909e/3d2049bb-024c-4c55-ac2e-c537e2a25c23"
-					(reference "#PWR058")
+					(reference "#PWR063")
 					(unit 1)
 				)
@@
 		(on_board yes)
 		(dnp no)
-		(property "Reference" "#PWR068"
+		(property "Reference" "#PWR073"
 			(at 194.31 147.32 0)
 			(effects
@@
 			(project "Icarus Flight Computer"
 				(path "/2a10c6de-1617-4216-ace2-cdde3ce2909e/3d2049bb-024c-4c55-ac2e-c537e2a25c23"
-					(reference "#PWR068")
+					(reference "#PWR073")
 					(unit 1)
 				)
@@
 		(dnp no)
 		(fields_autoplaced yes)
-		(property "Reference" "C24"
+		(property "Reference" "C25"
 			(at 229.87 59.6899 0)
 			(effects
@@
 			(project "Icarus Flight Computer"
 				(path "/2a10c6de-1617-4216-ace2-cdde3ce2909e/3d2049bb-024c-4c55-ac2e-c537e2a25c23"
-					(reference "C24")
+					(reference "C25")
 					(unit 1)
 				)
@@
 		(on_board yes)
 		(dnp no)
-		(property "Reference" "#PWR059"
+		(property "Reference" "#PWR064"
 			(at 167.64 77.47 0)
 			(effects
@@
 			(project "Icarus Flight Computer"
 				(path "/2a10c6de-1617-4216-ace2-cdde3ce2909e/3d2049bb-024c-4c55-ac2e-c537e2a25c23"
-					(reference "#PWR059")
+					(reference "#PWR064")
 					(unit 1)
 				)
@@
 		(on_board yes)
 		(dnp no)
-		(property "Reference" "#PWR053"
+		(property "Reference" "#PWR058"
 			(at 76.2 48.26 0)
 			(effects
@@
 			(project "Icarus Flight Computer"
 				(path "/2a10c6de-1617-4216-ace2-cdde3ce2909e/3d2049bb-024c-4c55-ac2e-c537e2a25c23"
-					(reference "#PWR053")
+					(reference "#PWR058")
 					(unit 1)
 				)
@@
 		(on_board yes)
 		(dnp no)
-		(property "Reference" "#PWR055"
+		(property "Reference" "#PWR060"
 			(at 109.22 57.15 0)
 			(effects
@@
 			(project "Icarus Flight Computer"
 				(path "/2a10c6de-1617-4216-ace2-cdde3ce2909e/3d2049bb-024c-4c55-ac2e-c537e2a25c23"
-					(reference "#PWR055")
+					(reference "#PWR060")
 					(unit 1)
 				)
@@
 		(on_board yes)
 		(dnp no)
-		(property "Reference" "#PWR064"
+		(property "Reference" "#PWR069"
 			(at 215.9 125.73 0)
 			(effects
@@
 			(project "Icarus Flight Computer"
 				(path "/2a10c6de-1617-4216-ace2-cdde3ce2909e/3d2049bb-024c-4c55-ac2e-c537e2a25c23"
-					(reference "#PWR064")
+					(reference "#PWR069")
 					(unit 1)
 				)
@@
 		(dnp no)
 		(fields_autoplaced yes)
-		(property "Reference" "C25"
+		(property "Reference" "C26"
 			(at 241.3 59.6899 0)
 			(effects
@@
 			(project "Icarus Flight Computer"
 				(path "/2a10c6de-1617-4216-ace2-cdde3ce2909e/3d2049bb-024c-4c55-ac2e-c537e2a25c23"
-					(reference "C25")
+					(reference "C26")
 					(unit 1)
 				)
@@
 		(dnp no)
 		(fields_autoplaced yes)
-		(property "Reference" "C29"
+		(property "Reference" "C30"
 			(at 132.08 128.2699 0)
 			(effects
@@
 			(project "Icarus Flight Computer"
 				(path "/2a10c6de-1617-4216-ace2-cdde3ce2909e/3d2049bb-024c-4c55-ac2e-c537e2a25c23"
-					(reference "C29")
+					(reference "C30")
 					(unit 1)
 				)
@@
 		(on_board yes)
 		(dnp no)
-		(property "Reference" "#PWR063"
+		(property "Reference" "#PWR068"
 			(at 194.31 119.38 0)
 			(effects
@@
 			(project "Icarus Flight Computer"
 				(path "/2a10c6de-1617-4216-ace2-cdde3ce2909e/3d2049bb-024c-4c55-ac2e-c537e2a25c23"
-					(reference "#PWR063")
+					(reference "#PWR068")
 					(unit 1)
 				)
@@
 		(dnp no)
 		(fields_autoplaced yes)
-		(property "Reference" "C23"
+		(property "Reference" "C24"
 			(at 218.44 59.6899 0)
 			(effects
@@
 			(project "Icarus Flight Computer"
 				(path "/2a10c6de-1617-4216-ace2-cdde3ce2909e/3d2049bb-024c-4c55-ac2e-c537e2a25c23"
-					(reference "C23")
+					(reference "C24")
 					(unit 1)
 				)
@@
 		(on_board yes)
 		(dnp no)
-		(property "Reference" "#PWR070"
+		(property "Reference" "#PWR075"
 			(at 87.63 149.86 0)
 			(effects
@@
 			(project "Icarus Flight Computer"
 				(path "/2a10c6de-1617-4216-ace2-cdde3ce2909e/3d2049bb-024c-4c55-ac2e-c537e2a25c23"
-					(reference "#PWR070")
+					(reference "#PWR075")
 					(unit 1)
 				)
@@
 		(on_board yes)
 		(dnp no)
-		(property "Reference" "#PWR056"
+		(property "Reference" "#PWR061"
 			(at 214.63 58.42 0)
 			(effects
@@
 			(project "Icarus Flight Computer"
 				(path "/2a10c6de-1617-4216-ace2-cdde3ce2909e/3d2049bb-024c-4c55-ac2e-c537e2a25c23"
-					(reference "#PWR056")
+					(reference "#PWR061")
 					(unit 1)
 				)
@@
 		(on_board yes)
 		(dnp no)
-		(property "Reference" "#PWR061"
+		(property "Reference" "#PWR066"
 			(at 182.88 81.28 0)
 			(effects
@@
 			(project "Icarus Flight Computer"
 				(path "/2a10c6de-1617-4216-ace2-cdde3ce2909e/3d2049bb-024c-4c55-ac2e-c537e2a25c23"
-					(reference "#PWR061")
+					(reference "#PWR066")
 					(unit 1)
 				)
@@
 		(on_board yes)
 		(dnp no)
-		(property "Reference" "#PWR057"
+		(property "Reference" "#PWR062"
 			(at 109.22 72.39 0)
 			(effects
@@
 			(project "Icarus Flight Computer"
 				(path "/2a10c6de-1617-4216-ace2-cdde3ce2909e/3d2049bb-024c-4c55-ac2e-c537e2a25c23"
-					(reference "#PWR057")
+					(reference "#PWR062")
 					(unit 1)
 				)
@@
 		(dnp no)
 		(fields_autoplaced yes)
-		(property "Reference" "C21"
+		(property "Reference" "C22"
 			(at 113.03 58.4199 0)
 			(effects
@@
 			(project "Icarus Flight Computer"
 				(path "/2a10c6de-1617-4216-ace2-cdde3ce2909e/3d2049bb-024c-4c55-ac2e-c537e2a25c23"
-					(reference "C21")
+					(reference "C22")
 					(unit 1)
 				)
