File: Schematic/GPS.kicad_sch (KiCad schematic)
At the start: 8 parts, among them J5 U.FL, U10 NEO-M9N-00B

Commit message: Made board smaller
Parts:
- D4: MPN C965812 -> C84256
- U10: MPN (none) -> C5119087
- renumbered C31 to C32, C32 to C33, J5 to J6
Changed lines of the file:
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@@
 		(title "Icarus Flight Computer")
 		(date "2025-04-30")
-		(rev "1.0")
+		(rev "V1.0")
 		(company "Daedalus Industries")
 		(comment 1 "Onboard flight computer for the Icarus rocket")
 		(comment 2 "GPS module for altitude and position correction/estimation ")
+		(comment 3 "Designer: Mattia Gregnanin")
 	)
 	(rectangle
@@
 		(on_board yes)
 		(dnp no)
-		(property "Reference" "#PWR073"
+		(property "Reference" "#PWR078"
 			(at 36.83 58.42 0)
 			(effects
@@
 			(project "Icarus Flight Computer"
 				(path "/2a10c6de-1617-4216-ace2-cdde3ce2909e/be8ac4a6-073a-4832-a49b-0d978579d155"
-					(reference "#PWR073")
+					(reference "#PWR078")
 					(unit 1)
 				)
@@
 		(on_board yes)
 		(dnp no)
-		(property "Reference" "#PWR072"
+		(property "Reference" "#PWR077"
 			(at 85.09 30.48 0)
 			(effects
@@
 			(project "Icarus Flight Computer"
 				(path "/2a10c6de-1617-4216-ace2-cdde3ce2909e/be8ac4a6-073a-4832-a49b-0d978579d155"
-					(reference "#PWR072")
+					(reference "#PWR077")
 					(unit 1)
 				)
@@
 		(dnp no)
 		(fields_autoplaced yes)
-		(property "Reference" "C31"
+		(property "Reference" "C32"
 			(at 40.64 59.6899 0)
 			(effects
@@
 			(project "Icarus Flight Computer"
 				(path "/2a10c6de-1617-4216-ace2-cdde3ce2909e/be8ac4a6-073a-4832-a49b-0d978579d155"
-					(reference "C31")
+					(reference "C32")
 					(unit 1)
 				)
@@
 		(on_board yes)
 		(dnp no)
-		(property "Reference" "#PWR075"
+		(property "Reference" "#PWR080"
 			(at 115.57 88.9 0)
 			(effects
@@
 			(project "Icarus Flight Computer"
 				(path "/2a10c6de-1617-4216-ace2-cdde3ce2909e/be8ac4a6-073a-4832-a49b-0d978579d155"
-					(reference "#PWR075")
+					(reference "#PWR080")
 					(unit 1)
 				)
@@
 			)
 		)
-		(property "MPN" "C965812"
+		(property "MPN" "C84256"
 			(at 109.22 69.85 0)
 			(effects
@@
 			)
 		)
+		(property "MPN" "C5119087"
+			(at 85.09 62.23 0)
+			(effects
+				(font
+					(size 1.27 1.27)
+				)
+				(hide yes)
+			)
+		)
 		(pin "21"
 		)
@@
 		(dnp no)
 		(fields_autoplaced yes)
-		(property "Reference" "C32"
+		(property "Reference" "C33"
 			(at 161.29 78.7399 0)
 			(effects
@@
 			(project "Icarus Flight Computer"
 				(path "/2a10c6de-1617-4216-ace2-cdde3ce2909e/be8ac4a6-073a-4832-a49b-0d978579d155"
-					(reference "C32")
+					(reference "C33")
 					(unit 1)
 				)
@@
 		(on_board yes)
 		(dnp no)
-		(property "Reference" "#PWR071"
+		(property "Reference" "#PWR076"
 			(at 80.01 40.64 0)
 			(effects
@@
 		(property "Description" "Power symbol creates a global label with name \"+3.3V\""
 			(at 80.01 36.83 0)
-			(effects
-				(font
-					(size 1.27 1.27)
-				)
-				(hide yes)
-			)
-		)
-		(pin "1"
-		)
-		(instances
-			(project "Icarus Flight Computer"
-				(path "/2a10c6de-1617-4216-ace2-cdde3ce2909e/be8ac4a6-073a-4832-a49b-0d978579d155"
-					(reference "#PWR071")
-					(unit 1)
-				)
-			)
-		)
-	)
-	(symbol
-		(lib_id "power:GND")
-		(at 157.48 86.36 0)
-		(unit 1)
-		(exclude_from_sim no)
-		(in_bom yes)
-		(on_board yes)
-		(dnp no)
-		(property "Reference" "#PWR076"
-			(at 157.48 92.71 0)
-			(effects
-				(font
-					(size 1.27 1.27)
-				)
-				(hide yes)
-			)
-		)
-		(property "Value" "GND"
-			(at 157.48 90.17 0)
-			(effects
-				(font
-					(size 1.27 1.27)
-				)
-			)
-		)
-		(property "Footprint" ""
-			(at 157.48 86.36 0)
-			(effects
-				(font
-					(size 1.27 1.27)
-				)
-				(hide yes)
-			)
-		)
-		(property "Datasheet" ""
-			(at 157.48 86.36 0)
-			(effects
-				(font
-					(size 1.27 1.27)
-				)
-				(hide yes)
-			)
-		)
-		(property "Description" "Power symbol creates a global label with name \"GND\" , ground"
-			(at 157.48 86.36 0)
 			(effects
 				(font
@@
 	(symbol
 		(lib_id "power:GND")
-		(at 85.09 87.63 0)
+		(at 157.48 86.36 0)
 		(unit 1)
 		(exclude_from_sim no)
@@
 		(on_board yes)
 		(dnp no)
-		(property "Reference" "#PWR078"
-			(at 85.09 93.98 0)
+		(property "Reference" "#PWR081"
+			(at 157.48 92.71 0)
 			(effects
 				(font
@@
 		)
 		(property "Value" "GND"
-			(at 85.09 91.44 0)
+			(at 157.48 90.17 0)
 			(effects
 				(font
@@
 		)
 		(property "Footprint" ""
-			(at 85.09 87.63 0)
+			(at 157.48 86.36 0)
 			(effects
 				(font
@@
 		)
 		(property "Datasheet" ""
-			(at 85.09 87.63 0)
+			(at 157.48 86.36 0)
 			(effects
 				(font
@@
 		)
 		(property "Description" "Power symbol creates a global label with name \"GND\" , ground"
-			(at 85.09 87.63 0)
+			(at 157.48 86.36 0)
 			(effects
 				(font
@@
 			(project "Icarus Flight Computer"
 				(path "/2a10c6de-1617-4216-ace2-cdde3ce2909e/be8ac4a6-073a-4832-a49b-0d978579d155"
-					(reference "#PWR078")
+					(reference "#PWR081")
+					(unit 1)
+				)
+			)
+		)
+	)
+	(symbol
+		(lib_id "power:GND")
+		(at 85.09 87.63 0)
+		(unit 1)
+		(exclude_from_sim no)
+		(in_bom yes)
+		(on_board yes)
+		(dnp no)
+		(property "Reference" "#PWR083"
+			(at 85.09 93.98 0)
+			(effects
+				(font
+					(size 1.27 1.27)
+				)
+				(hide yes)
+			)
+		)
+		(property "Value" "GND"
+			(at 85.09 91.44 0)
+			(effects
+				(font
+					(size 1.27 1.27)
+				)
+			)
+		)
+		(property "Footprint" ""
+			(at 85.09 87.63 0)
+			(effects
+				(font
+					(size 1.27 1.27)
+				)
+				(hide yes)
+			)
+		)
+		(property "Datasheet" ""
+			(at 85.09 87.63 0)
+			(effects
+				(font
+					(size 1.27 1.27)
+				)
+				(hide yes)
+			)
+		)
+		(property "Description" "Power symbol creates a global label with name \"GND\" , ground"
+			(at 85.09 87.63 0)
+			(effects
+				(font
+					(size 1.27 1.27)
+				)
+				(hide yes)
+			)
+		)
+		(pin "1"
+		)
+		(instances
+			(project "Icarus Flight Computer"
+				(path "/2a10c6de-1617-4216-ace2-cdde3ce2909e/be8ac4a6-073a-4832-a49b-0d978579d155"
+					(reference "#PWR083")
 					(unit 1)
 				)
@@
 		(dnp no)
 		(fields_autoplaced yes)
-		(property "Reference" "J5"
+		(property "Reference" "J6"
 			(at 170.18 62.5231 0)
 			(effects
@@
 			(project ""
 				(path "/2a10c6de-1617-4216-ace2-cdde3ce2909e/be8ac4a6-073a-4832-a49b-0d978579d155"
-					(reference "J5")
+					(reference "J6")
 					(unit 1)
 				)
@@
 		(on_board yes)
 		(dnp no)
-		(property "Reference" "#PWR074"
+		(property "Reference" "#PWR079"
 			(at 36.83 73.66 0)
 			(effects
@@
 			(project "Icarus Flight Computer"
 				(path "/2a10c6de-1617-4216-ace2-cdde3ce2909e/be8ac4a6-073a-4832-a49b-0d978579d155"
-					(reference "#PWR074")
+					(reference "#PWR079")
 					(unit 1)
 				)
@@
 		(on_board yes)
 		(dnp no)
-		(property "Reference" "#PWR077"
+		(property "Reference" "#PWR082"
 			(at 167.64 92.71 0)
 			(effects
@@
 			(project "Icarus Flight Computer"
 				(path "/2a10c6de-1617-4216-ace2-cdde3ce2909e/be8ac4a6-073a-4832-a49b-0d978579d155"
-					(reference "#PWR077")
+					(reference "#PWR082")
 					(unit 1)
 				)

Commit message: V1.0
Parts:
- J5: renamed from J6; value U.FL -> SMA; footprint Connector_Coaxial:U.FL_Hirose_U.FL-R-SMT-1_Vertical -> Connector_Coaxial:SMA_Amphenol_132134_Vertical; MPN C5137195 -> C3174425
- R17: renamed from R13; MPN C17903 -> C25349
- renumbered C32 to C33, C33 to C34, R14 to R18
Other:
- note added: "4mA max"
