File: Schematic/MCU.kicad_sch (KiCad schematic)
At the start: 29 parts, among them J1 Conn_01x04_Socket, J2 JST PH 2.0, SW1 SW_Push, U1 STM32F405RGT6, U2 W25Q128JVP, Y1 16MHz

Commit message: Added Docs folder
Connections:
- net GND: now also J2.1 (Pin_1); no longer J2.5 (Pin_5)
- net SERVO1_PWM: now also J2.2 (Pin_2); no longer J2.1 (Pin_1)
- net SERVO2_PWM: now also J2.3 (Pin_3); no longer J2.2 (Pin_2)
- net SERVO3_PWM: now also J2.4 (Pin_4); no longer J2.3 (Pin_3)
- net SERVO4_PWM: now also J2.5 (Pin_5); no longer J2.4 (Pin_4)
Other:
- moved on the sheet: J2
Changed lines of the file:
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@@
 	(text "Servo Connector"
 		(exclude_from_sim no)
-		(at 149.86 127 0)
+		(at 149.86 126.238 0)
 		(effects
 			(font
@@
 	(text "Used to drive 4 servos"
 		(exclude_from_sim no)
-		(at 148.336 155.448 0)
+		(at 149.86 155.448 0)
 		(effects
 			(font
@@
 	(wire
 		(pts
-			(xy 147.32 137.16) (xy 149.86 137.16)
+			(xy 59.69 48.26) (xy 48.26 48.26)
 		)
 		(stroke
@@
 	(wire
 		(pts
-			(xy 59.69 48.26) (xy 48.26 48.26)
+			(xy 87.63 134.62) (xy 99.06 134.62)
 		)
 		(stroke
@@
 	(wire
 		(pts
-			(xy 87.63 134.62) (xy 99.06 134.62)
+			(xy 59.69 46.99) (xy 59.69 48.26)
 		)
 		(stroke
@@
 	(wire
 		(pts
-			(xy 59.69 46.99) (xy 59.69 48.26)
+			(xy 210.82 121.92) (xy 210.82 119.38)
 		)
 		(stroke
@@
 	(wire
 		(pts
-			(xy 210.82 121.92) (xy 210.82 119.38)
+			(xy 59.69 38.1) (xy 71.12 38.1)
 		)
 		(stroke
@@
 	(wire
 		(pts
-			(xy 59.69 38.1) (xy 71.12 38.1)
+			(xy 147.32 138.43) (xy 149.86 138.43)
 		)
 		(stroke
@@
 	(wire
 		(pts
-			(xy 147.32 142.24) (xy 149.86 142.24)
-		)
-		(stroke
-			(width 0)
-			(type default)
-		)
-	)
-	(wire
-		(pts
 			(xy 214.63 99.06) (xy 217.17 99.06)
 		)
@@
 	(wire
 		(pts
+			(xy 147.32 143.51) (xy 149.86 143.51)
+		)
+		(stroke
+			(width 0)
+			(type default)
+		)
+	)
+	(wire
+		(pts
 			(xy 52.07 86.36) (xy 54.61 86.36)
 		)
@@
 	(wire
 		(pts
-			(xy 147.32 134.62) (xy 149.86 134.62)
-		)
-		(stroke
-			(width 0)
-			(type default)
-		)
-	)
-	(wire
-		(pts
 			(xy 86.36 146.05) (xy 88.9 146.05)
 		)
@@
 	(wire
 		(pts
-			(xy 149.86 144.78) (xy 147.32 144.78)
+			(xy 48.26 38.1) (xy 36.83 38.1)
 		)
 		(stroke
@@
 	(wire
 		(pts
-			(xy 48.26 38.1) (xy 36.83 38.1)
+			(xy 260.35 129.54) (xy 257.81 129.54)
 		)
 		(stroke
@@
 	(wire
 		(pts
-			(xy 260.35 129.54) (xy 257.81 129.54)
+			(xy 191.77 119.38) (xy 191.77 121.92)
 		)
 		(stroke
@@
 	(wire
 		(pts
-			(xy 191.77 119.38) (xy 191.77 121.92)
+			(xy 132.08 46.99) (xy 132.08 48.26)
 		)
 		(stroke
@@
 	(wire
 		(pts
-			(xy 147.32 139.7) (xy 149.86 139.7)
+			(xy 54.61 147.32) (xy 54.61 149.86)
 		)
 		(stroke
@@
 	(wire
 		(pts
-			(xy 132.08 46.99) (xy 132.08 48.26)
+			(xy 149.86 135.89) (xy 147.32 135.89)
 		)
 		(stroke
@@
 	(wire
 		(pts
-			(xy 54.61 147.32) (xy 54.61 149.86)
+			(xy 147.32 146.05) (xy 149.86 146.05)
 		)
 		(stroke
@@
 	(wire
 		(pts
-			(xy 147.32 144.78) (xy 147.32 147.32)
+			(xy 217.17 116.84) (xy 200.66 116.84)
 		)
 		(stroke
@@
 	(wire
 		(pts
-			(xy 217.17 116.84) (xy 200.66 116.84)
+			(xy 26.67 96.52) (xy 26.67 99.06)
 		)
 		(stroke
@@
 	(wire
 		(pts
-			(xy 26.67 96.52) (xy 26.67 99.06)
+			(xy 210.82 129.54) (xy 210.82 132.08)
 		)
 		(stroke
@@
 	(wire
 		(pts
-			(xy 210.82 129.54) (xy 210.82 132.08)
+			(xy 86.36 148.59) (xy 88.9 148.59)
 		)
 		(stroke
@@
 	(wire
 		(pts
-			(xy 86.36 148.59) (xy 88.9 148.59)
+			(xy 147.32 135.89) (xy 147.32 134.62)
+		)
+		(stroke
+			(width 0)
+			(type default)
+		)
+	)
+	(wire
+		(pts
+			(xy 147.32 140.97) (xy 149.86 140.97)
 		)
 		(stroke
@@
 		)
 	)
-	(global_label "SERVO4_PWM"
-		(shape input)
-		(at 147.32 142.24 180)
-		(fields_autoplaced yes)
-		(effects
-			(font
-				(size 1.27 1.27)
-			)
-			(justify right)
-		)
-		(property "Intersheetrefs" "${INTERSHEET_REFS}"
-			(at 131.9373 142.24 0)
-			(effects
-				(font
-					(size 1.27 1.27)
-				)
-				(justify right)
-				(hide yes)
-			)
-		)
-	)
 	(global_label "SWCLK"
 		(shape input)
@@
 		)
 	)
-	(global_label "SERVO1_PWM"
-		(shape input)
-		(at 147.32 134.62 180)
-		(fields_autoplaced yes)
-		(effects
-			(font
-				(size 1.27 1.27)
-			)
-			(justify right)
-		)
-		(property "Intersheetrefs" "${INTERSHEET_REFS}"
-			(at 131.9373 134.62 0)
-			(effects
-				(font
-					(size 1.27 1.27)
-				)
-				(justify right)
-				(hide yes)
-			)
-		)
-	)
 	(global_label "FLASH_SPI_SCK"
 		(shape output)
@@
 		)
 	)
-	(global_label "SERVO3_PWM"
-		(shape input)
-		(at 147.32 139.7 180)
-		(fields_autoplaced yes)
-		(effects
-			(font
-				(size 1.27 1.27)
-			)
-			(justify right)
-		)
-		(property "Intersheetrefs" "${INTERSHEET_REFS}"
-			(at 131.9373 139.7 0)
-			(effects
-				(font
-					(size 1.27 1.27)
-				)
-				(justify right)
-				(hide yes)
-			)
-		)
-	)
 	(global_label "RF_UART_RX"
 		(shape output)
@@
 		)
 	)
+	(global_label "SERVO1_PWM"
+		(shape input)
+		(at 147.32 138.43 180)
+		(fields_autoplaced yes)
+		(effects
+			(font
+				(size 1.27 1.27)
+			)
+			(justify right)
+		)
+		(property "Intersheetrefs" "${INTERSHEET_REFS}"
+			(at 131.9373 138.43 0)
+			(effects
+				(font
+					(size 1.27 1.27)
+				)
+				(justify right)
+				(hide yes)
+			)
+		)
+	)
 	(global_label "GPS_UART_RX"
 		(shape input)
@@
 		)
 	)
+	(global_label "SERVO2_PWM"
+		(shape input)
+		(at 147.32 140.97 180)
+		(fields_autoplaced yes)
+		(effects
+			(font
+				(size 1.27 1.27)
+			)
+			(justify right)
+		)
+		(property "Intersheetrefs" "${INTERSHEET_REFS}"
+			(at 131.9373 140.97 0)
+			(effects
+				(font
+					(size 1.27 1.27)
+				)
+				(justify right)
+				(hide yes)
+			)
+		)
+	)
+	(global_label "SERVO4_PWM"
+		(shape input)
+		(at 147.32 146.05 180)
+		(fields_autoplaced yes)
+		(effects
+			(font
+				(size 1.27 1.27)
+			)
+			(justify right)
+		)
+		(property "Intersheetrefs" "${INTERSHEET_REFS}"
+			(at 131.9373 146.05 0)
+			(effects
+				(font
+					(size 1.27 1.27)
+				)
+				(justify right)
+				(hide yes)
+			)
+		)
+	)
 	(global_label "USB_D-"
 		(shape bidirectional)
@@
 		)
 	)
-	(global_label "SERVO2_PWM"
+	(global_label "SERVO3_PWM"
 		(shape input)
-		(at 147.32 137.16 180)
+		(at 147.32 143.51 180)
 		(fields_autoplaced yes)
 		(effects
@@
 		)
 		(property "Intersheetrefs" "${INTERSHEET_REFS}"
-			(at 131.9373 137.16 0)
+			(at 131.9373 143.51 0)
 			(effects
 				(font
@@
 	(symbol
 		(lib_id "Connector_Generic:Conn_01x05")
-		(at 154.94 139.7 0)
+		(at 154.94 140.97 0)
 		(unit 1)
 		(exclude_from_sim no)
@@
 		(dnp no)
 		(property "Reference" "J2"
-			(at 156.972 147.066 0)
+			(at 156.21 133.604 0)
 			(effects
 				(font
@@
 		)
 		(property "Value" "JST PH 2.0"
-			(at 156.21 131.826 0)
+			(at 156.21 148.336 0)
 			(effects
 				(font
@@
 		)
 		(property "Footprint" "Connector_JST:JST_PH_S5B-PH-K_1x05_P2.00mm_Horizontal"
-			(at 154.94 139.7 0)
+			(at 154.94 140.97 0)
 			(effects
 				(font
@@
 		)
 		(property "Datasheet" "~"
-			(at 154.94 139.7 0)
+			(at 154.94 140.97 0)
 			(effects
 				(font
@@
 		)
 		(property "Description" "Generic connector, single row, 01x05, script generated (kicad-library-utils/schlib/autogen/connector/)"
-			(at 154.94 139.7 0)
+			(at 154.94 140.97 0)
 			(effects
 				(font
@@
 		)
 		(property "MPN" "C265085"
-			(at 154.94 139.7 0)
+			(at 154.94 140.97 0)
 			(effects
 				(font
@@
 	(symbol
 		(lib_id "power:GND")
-		(at 147.32 147.32 0)
+		(at 147.32 134.62 0)
+		(mirror x)
 		(unit 1)
 		(exclude_from_sim no)
@@
 		(dnp no)
 		(property "Reference" "#PWR031"
-			(at 147.32 153.67 0)
+			(at 147.32 128.27 0)
 			(effects
 				(font
@@
 		)
 		(property "Value" "GND"
-			(at 147.32 151.13 0)
+			(at 147.32 130.81 0)
 			(effects
 				(font
@@
 		)
 		(property "Footprint" ""
-			(at 147.32 147.32 0)
+			(at 147.32 134.62 0)
 			(effects
 				(font
@@
 		)
 		(property "Datasheet" ""
-			(at 147.32 147.32 0)
+			(at 147.32 134.62 0)
 			(effects
 				(font
@@
 		)
 		(property "Description" "Power symbol creates a global label with name \"GND\" , ground"
-			(at 147.32 147.32 0)
+			(at 147.32 134.62 0)
 			(effects
 				(font

Commit message: Made board smaller
Parts:
- removed R5, R6: 2k, Resistor_SMD:R_0402_1005Metric, symbol Device:R
- added C16: 100n, Capacitor_SMD:C_0402_1005Metric, symbol Device:C
- added R2: 10k, Resistor_SMD:R_0402_1005Metric, symbol Device:R
- D1: MPN C965812 -> C84256
- J1: value Conn_01x04_Socket -> Conn_01x04_Pin; footprint Connector_PinSocket_2.54mm:PinSocket_1x04_P2.54mm_Vertical -> Connector_PinHeader_2.54mm:PinHeader_1x04_P2.54mm_Vertical; symbol Connector:Conn_01x04_Socket -> Connector:Conn_01x04_Pin; MPN C2718488 -> C2691448
- J2: footprint Connector_JST:JST_PH_S5B-PH-K_1x05_P2.00mm_Horizontal -> Connector_JST:JST_PH_B5B-PH-K_1x05_P2.00mm_Vertical; MPN C265085 -> C5359602
- U2: value W25Q128JVP -> W25Q128JVSIQ; MPN (none) -> C97521
- renumbered C13 to C11, C11 to C12, C12 to C13, R2 to R3, R3 to R4, R4 to R5
Connections:
- net +3.3V: now also C16.1
- net ACC_INT: now also U1.27 (PB1); no longer U1.28 (PB2)
- net GND: now also J2.5 (Pin_5), C16.2, R2.2; no longer J2.1 (Pin_1)
- net PYRO_A_FIRE: now also U1.4 (PC15); no longer U1.3 (PC14)
- net PYRO_B_FIRE: now also U1.3 (PC14); no longer U1.4 (PC15)
- net SERVO1_PWM: now also J2.4 (Pin_4); no longer J2.2 (Pin_2)
- net SERVO3_PWM: now also J2.2 (Pin_2); no longer J2.4 (Pin_4)
- net SERVO4_PWM: now also J2.1 (Pin_1); no longer J2.5 (Pin_5)
- new net BOOT1: R2.1, U1.28 (PB2)
- no-connect marks 13 -> 12
Other:
- note added: "BOOT Pins"
- note added: "I2C Pullup Resistors"
- note removed: "BOOT0 Switch"
- note removed: "Enable firmware flashing from USB (i.e. for Arduino)"
- note removed: "I2C Pullup Resistor"
- moved on the sheet: C10, C11, C12, C13, J2, R4, R5, U2, Y1

Commit message: V1.0
Parts:
- removed C11: 100n, Capacitor_SMD:C_0402_1005Metric, symbol Device:C
- removed J2: JST PH 2.0, Connector_JST:JST_PH_B5B-PH-K_1x05_P2.00mm_Vertical, symbol Connector_Generic:Conn_01x05
- added R1, R2: 22R, Resistor_SMD:R_0402_1005Metric, symbol Device:R
- added R8, R9: 2k, Resistor_SMD:R_0402_1005Metric, symbol Device:R
- renumbered C12 to C11, C13 to C12, C14 to C13, C15 to C14, C16 to C15, R1 to R3, R2 to R4, R3 to R5, R4 to R6, R5 to R7
Connections:
- net MAG_CS is gone; now on net IMU_CS: U1.37 (PC6)
- net +3.3V: now also R8.1, R9.1
- net IMU_CS: no longer U1.38 (PC7)
- net IMU_INT: now also U1.38 (PC7); no longer U1.39 (PC8)
- net MAG_I2C_SDA: now reaches U1.40 (PC9)
- net MAG_I2C_SDA: now also R9.2
- net MAG_I2C_SCL: now reaches U1.41 (PA8)
- net MAG_I2C_SCL: now also R8.2
- net SWCLK renamed SW_CLK
- net SW_CLK: now also R2.1; no longer J1.3 (Pin_3)
- net SWDIO renamed SW_DIO
- net SW_DIO: now also R1.1; no longer J1.2 (Pin_2)
- new net SW_CLK_HEADER: J1.3 (Pin_3), R2.2
- new net SW_DIO_HEADER: J1.2 (Pin_2), R1.2
- no-connect marks 12 -> 11
Other:
- note added: "GPS has internal pull-up resistors"
- note removed: "Servo Connector"
- note removed: "Used to drive 4 servos"
- moved on the sheet: C1, C11, C12, C15, C2, C3, C4, C5, C6, C7, C8, C9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
