File: Schematic/Power.kicad_sch (KiCad schematic)
At the start: 15 parts, among them J4 JST PH 2.0, Q1 DMG2305UX, U4 TPS3839G33DBZ, U5 TPS631000

Commit message: Made board smaller
Parts:
- removed U4: TPS3839G33DBZ, Package_TO_SOT_SMD:SOT-23, symbol Power_Supervisor:TPS3839DBZ
- added J5: Conn_01x02_Pin, Connector_PinHeader_2.54mm:PinHeader_1x02_P2.54mm_Vertical, symbol Connector:Conn_01x02_Pin
- added U4: TPS3831G33DQNR, Package_SON:Texas_X2SON-4_1x1mm_P0.65mm, symbol Power_Supervisor:TPS3831
- D2: MPN C965812 -> C84256
- D3: MPN (none) -> C47460
- J4: MPN C131337 -> C2683610
- renumbered C17 to C19, C19 to C20, C20 to C21
Connections:
- net +3.3V: now also U4.4 (VDD)
- net GND: now also J4.1 (Pin_1), J5.2 (Pin_2), U4.3 (GND), U4.5 (TP); no longer J4.2 (Pin_2)
- net VBAT: now also J4.2 (Pin_2); no longer J4.1 (Pin_1)
- net ~{RESET}: now also U4.1 (~{RESET})
- new net ~{MR}: J5.1 (Pin_1), U4.2 (~{MR})
Other:
- note added: "Keep MCU resetted until 3.08V are achieved"
- note removed: "Keep MCU resetted until 3.08V"
- moved on the sheet: C18, C19, C20, C21, D2, D3, J4, L1, Q1, R10, R11, R12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

Commit message: V1.0
Parts:
- Q1: symbol Transistor_FET:DMG2305UX -> My_Transistor:DMG2305UX
- R16: renamed from R12; value 10k -> 100k; MPN C25531 -> C25741
- U5: symbol Regulator_Switching:TPS631000 -> My_Regulator:TPS631000
- renumbered C18 to C17, C19 to C18, C20 to C19, C21 to C20, J4 to J3, J5 to J4, R9 to R13, R10 to R14, R11 to R15
Other:
- moved on the sheet: C17, C18, J3, J4, U4
