File: Schematic/Pyro.kicad_sch (KiCad schematic)
At the start: 11 parts, among them J6 Screw_Terminal_01x06, Q2 Si7232DN

Commit message: Made board smaller
Parts:
- J7: renamed from J6; footprint TerminalBlock_Phoenix:TerminalBlock_Phoenix_MKDS-1,5-6-5.08_1x06_P5.08mm_Horizontal -> TerminalBlock_Phoenix:TerminalBlock_Phoenix_MPT-0,5-6-2.54_1x06_P2.54mm_Horizontal; MPN C69810 -> C3817456
- Q2: MPN (none) -> C144854
- renumbered C35 to C36
Connections:
- net GND: now also J7.5 (Pin_5); no longer J7.2 (Pin_2)
- net PYRO_A: now also J7.3 (Pin_3); no longer J7.4 (Pin_4)
- net PYRO_B: now also J7.1 (Pin_1); no longer J7.6 (Pin_6)
- net PYRO_VBAT: now also J7.2 (Pin_2), J7.4 (Pin_4), J7.6 (Pin_6); no longer J7.1 (Pin_1), J7.3 (Pin_3), J7.5 (Pin_5)
Changed lines of the file:
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@@
 		(title "Icarus Flight Computer")
 		(date "2025-04-30")
-		(rev "1.0")
+		(rev "V1.0")
 		(company "Daedalus Industries")
 		(comment 1 "Onboard flight computer for the Icarus rocket")
 		(comment 2 "E-match firing for chutes")
+		(comment 3 "Designer: Mattia Gregnanin")
 	)
 	(rectangle
@@
 		(on_board yes)
 		(dnp no)
-		(property "Reference" "#PWR085"
+		(property "Reference" "#PWR090"
 			(at 95.25 55.88 0)
 			(effects
@@
 			(project "Icarus Flight Computer"
 				(path "/2a10c6de-1617-4216-ace2-cdde3ce2909e/550d7cb8-eef1-4026-bc63-2e74eac34178"
-					(reference "#PWR085")
+					(reference "#PWR090")
 					(unit 1)
 				)
@@
 		(on_board yes)
 		(dnp no)
-		(property "Reference" "#PWR086"
+		(property "Reference" "#PWR091"
 			(at 134.62 54.61 0)
 			(effects
@@
 			(project "Icarus Flight Computer"
 				(path "/2a10c6de-1617-4216-ace2-cdde3ce2909e/550d7cb8-eef1-4026-bc63-2e74eac34178"
-					(reference "#PWR086")
+					(reference "#PWR091")
 					(unit 1)
 				)
@@
 		(on_board yes)
 		(dnp no)
-		(property "Reference" "#PWR089"
+		(property "Reference" "#PWR094"
 			(at 55.88 95.25 0)
 			(effects
@@
 		(property "Description" "Power symbol creates a global label with name \"GND\" , ground"
 			(at 55.88 88.9 0)
+			(effects
+				(font
+					(size 1.27 1.27)
+				)
+				(hide yes)
+			)
+		)
+		(pin "1"
+		)
+		(instances
+			(project "Icarus Flight Computer"
+				(path "/2a10c6de-1617-4216-ace2-cdde3ce2909e/550d7cb8-eef1-4026-bc63-2e74eac34178"
+					(reference "#PWR094")
+					(unit 1)
+				)
+			)
+		)
+	)
+	(symbol
+		(lib_id "power:GND")
+		(at 76.2 49.53 0)
+		(unit 1)
+		(exclude_from_sim no)
+		(in_bom yes)
+		(on_board yes)
+		(dnp no)
+		(property "Reference" "#PWR089"
+			(at 76.2 55.88 0)
+			(effects
+				(font
+					(size 1.27 1.27)
+				)
+				(hide yes)
+			)
+		)
+		(property "Value" "GND"
+			(at 76.2 53.34 0)
+			(effects
+				(font
+					(size 1.27 1.27)
+				)
+			)
+		)
+		(property "Footprint" ""
+			(at 76.2 49.53 0)
+			(effects
+				(font
+					(size 1.27 1.27)
+				)
+				(hide yes)
+			)
+		)
+		(property "Datasheet" ""
+			(at 76.2 49.53 0)
+			(effects
+				(font
+					(size 1.27 1.27)
+				)
+				(hide yes)
+			)
+		)
+		(property "Description" "Power symbol creates a global label with name \"GND\" , ground"
+			(at 76.2 49.53 0)
 			(effects
 				(font
@@
 	(symbol
 		(lib_id "power:GND")
-		(at 76.2 49.53 0)
+		(at 149.86 73.66 0)
 		(unit 1)
 		(exclude_from_sim no)
@@
 		(on_board yes)
 		(dnp no)
-		(property "Reference" "#PWR084"
-			(at 76.2 55.88 0)
+		(property "Reference" "#PWR093"
+			(at 149.86 80.01 0)
 			(effects
 				(font
@@
 		)
 		(property "Value" "GND"
-			(at 76.2 53.34 0)
+			(at 149.86 77.47 0)
 			(effects
 				(font
@@
 		)
 		(property "Footprint" ""
-			(at 76.2 49.53 0)
+			(at 149.86 73.66 0)
 			(effects
 				(font
@@
 		)
 		(property "Datasheet" ""
-			(at 76.2 49.53 0)
+			(at 149.86 73.66 0)
 			(effects
 				(font
@@
 		)
 		(property "Description" "Power symbol creates a global label with name \"GND\" , ground"
-			(at 76.2 49.53 0)
+			(at 149.86 73.66 0)
 			(effects
 				(font
@@
 			(project "Icarus Flight Computer"
 				(path "/2a10c6de-1617-4216-ace2-cdde3ce2909e/550d7cb8-eef1-4026-bc63-2e74eac34178"
-					(reference "#PWR084")
-					(unit 1)
-				)
-			)
-		)
-	)
-	(symbol
-		(lib_id "power:GND")
-		(at 149.86 73.66 0)
-		(unit 1)
-		(exclude_from_sim no)
-		(in_bom yes)
-		(on_board yes)
-		(dnp no)
-		(property "Reference" "#PWR088"
-			(at 149.86 80.01 0)
-			(effects
-				(font
-					(size 1.27 1.27)
-				)
-				(hide yes)
-			)
-		)
-		(property "Value" "GND"
-			(at 149.86 77.47 0)
-			(effects
-				(font
-					(size 1.27 1.27)
-				)
-			)
-		)
-		(property "Footprint" ""
-			(at 149.86 73.66 0)
-			(effects
-				(font
-					(size 1.27 1.27)
-				)
-				(hide yes)
-			)
-		)
-		(property "Datasheet" ""
-			(at 149.86 73.66 0)
-			(effects
-				(font
-					(size 1.27 1.27)
-				)
-				(hide yes)
-			)
-		)
-		(property "Description" "Power symbol creates a global label with name \"GND\" , ground"
-			(at 149.86 73.66 0)
-			(effects
-				(font
-					(size 1.27 1.27)
-				)
-				(hide yes)
-			)
-		)
-		(pin "1"
-		)
-		(instances
-			(project "Icarus Flight Computer"
-				(path "/2a10c6de-1617-4216-ace2-cdde3ce2909e/550d7cb8-eef1-4026-bc63-2e74eac34178"
-					(reference "#PWR088")
+					(reference "#PWR093")
 					(unit 1)
 				)
@@
 		(on_board yes)
 		(dnp no)
-		(property "Reference" "#PWR091"
+		(property "Reference" "#PWR096"
 			(at 95.25 95.25 0)
 			(effects
@@
 			(project "Icarus Flight Computer"
 				(path "/2a10c6de-1617-4216-ace2-cdde3ce2909e/550d7cb8-eef1-4026-bc63-2e74eac34178"
-					(reference "#PWR091")
+					(reference "#PWR096")
 					(unit 1)
 				)
@@
 		(on_board yes)
 		(dnp no)
-		(property "Reference" "#PWR083"
+		(property "Reference" "#PWR088"
 			(at 55.88 55.88 0)
 			(effects
@@
 			(project "Icarus Flight Computer"
 				(path "/2a10c6de-1617-4216-ace2-cdde3ce2909e/550d7cb8-eef1-4026-bc63-2e74eac34178"
-					(reference "#PWR083")
+					(reference "#PWR088")
 					(unit 1)
 				)
@@
 	(symbol
 		(lib_id "Connector:Screw_Terminal_01x06")
-		(at 158.75 63.5 0)
+		(at 158.75 66.04 0)
+		(mirror x)
 		(unit 1)
 		(exclude_from_sim no)
@@
 		(on_board yes)
 		(dnp no)
-		(property "Reference" "J6"
-			(at 159.766 55.626 0)
+		(property "Reference" "J7"
+			(at 159.766 73.914 0)
 			(effects
 				(font
@@
 		)
 		(property "Value" "Screw_Terminal_01x06"
-			(at 159.258 74.168 0)
+			(at 159.258 55.372 0)
 			(effects
 				(font
@@
 			)
 		)
-		(property "Footprint" "TerminalBlock_Phoenix:TerminalBlock_Phoenix_MKDS-1,5-6-5.08_1x06_P5.08mm_Horizontal"
-			(at 158.75 63.5 0)
+		(property "Footprint" "TerminalBlock_Phoenix:TerminalBlock_Phoenix_MPT-0,5-6-2.54_1x06_P2.54mm_Horizontal"
+			(at 158.75 66.04 0)
 			(effects
 				(font
@@
 		)
 		(property "Datasheet" "~"
-			(at 158.75 63.5 0)
+			(at 158.75 66.04 0)
 			(effects
 				(font
@@
 		)
 		(property "Description" "Generic screw terminal, single row, 01x06, script generated (kicad-library-utils/schlib/autogen/connector/)"
-			(at 158.75 63.5 0)
-			(effects
-				(font
-					(size 1.27 1.27)
-				)
-				(hide yes)
-			)
-		)
-		(property "MPN" "C69810"
-			(at 158.75 63.5 0)
+			(at 158.75 66.04 0)
+			(effects
+				(font
+					(size 1.27 1.27)
+				)
+				(hide yes)
+			)
+		)
+		(property "MPN" "C3817456"
+			(at 158.75 66.04 0)
 			(effects
 				(font
@@
 			(project "Icarus Flight Computer"
 				(path "/2a10c6de-1617-4216-ace2-cdde3ce2909e/550d7cb8-eef1-4026-bc63-2e74eac34178"
-					(reference "J6")
+					(reference "J7")
 					(unit 1)
 				)
@@
 		(on_board yes)
 		(dnp no)
-		(property "Reference" "#PWR090"
+		(property "Reference" "#PWR095"
 			(at 76.2 95.25 0)
 			(effects
@@
 			(project "Icarus Flight Computer"
 				(path "/2a10c6de-1617-4216-ace2-cdde3ce2909e/550d7cb8-eef1-4026-bc63-2e74eac34178"
-					(reference "#PWR090")
+					(reference "#PWR095")
 					(unit 1)
 				)
@@
 		(dnp no)
 		(fields_autoplaced yes)
-		(property "Reference" "C35"
+		(property "Reference" "C36"
 			(at 138.43 57.1499 0)
 			(effects
@@
 			(project "Icarus Flight Computer"
 				(path "/2a10c6de-1617-4216-ace2-cdde3ce2909e/550d7cb8-eef1-4026-bc63-2e74eac34178"
-					(reference "C35")
+					(reference "C36")
 					(unit 1)
 				)
@@
 			)
 		)
+		(property "MPN" "C144854"
+			(at 73.66 36.83 0)
+			(effects
+				(font
+					(size 1.27 1.27)
+				)
+				(hide yes)
+			)
+		)
 		(pin "6"
 		)
@@
 		(on_board yes)
 		(dnp no)
-		(property "Reference" "#PWR087"
+		(property "Reference" "#PWR092"
 			(at 134.62 71.12 0)
 			(effects
@@
 			(project "Icarus Flight Computer"
 				(path "/2a10c6de-1617-4216-ace2-cdde3ce2909e/550d7cb8-eef1-4026-bc63-2e74eac34178"
-					(reference "#PWR087")
+					(reference "#PWR092")
 					(unit 1)
 				)
@@
 			(at 73.66 76.2 0)
 			(effects
+				(font
+					(size 1.27 1.27)
+				)
+				(hide yes)
+			)
+		)
+		(property "MPN" "C144854"
+			(at 73.66 76.2 0)
+			(effects

Commit message: V1.0
Parts:
- Q2: symbol Transistor_FET:Si7232DN -> My_Transistor:Si7232DN
- renumbered C36 to C37, J7 to J6, R15 to R19, R16 to R20, R17 to R21, R18 to R22, R19 to R23, R20 to R24, R21 to R25, R22 to R26
Other:
- moved on the sheet: C37, J6
