File: Schematic/Sensors.kicad_sch (KiCad schematic)
At the start: 14 parts, among them U6 ICM-45686, U7 ADXL375, U8 LIS2MDL, U9 MS5607-02BA

Commit message: V1.0
Parts:
- removed C28: 1u, Capacitor_SMD:C_0603_1608Metric, symbol Device:C
- added C26, C27: 100n, Capacitor_SMD:C_0402_1005Metric, symbol Device:C
- added C29: 10u, Capacitor_SMD:C_0805_2012Metric, symbol Device:C
- U6: symbol Sensor_Motion:ICM-45686 -> My_Sensor:ICM-45686
- U7: symbol Sensor_Motion:ADXL375 -> My_Sensor:ADXL375
- U9: footprint Package_LGA:LGA-8_3x5mm_P1.25mm -> My_Sensor:MS5607-02BA03
- renumbered C22 to C21, C23 to C22, C24 to C23, C25 to C24, C26 to C25, C27 to C28, C29 to C30, C30 to C31, C31 to C32
Connections:
- net MAG_CS is gone; now on net +3.3V: U8.3 (~{CS})
- net +3.3V: now also C26.1, C27.1, C29.1
- net GND: now also C26.2, C27.2, C29.2
- net SPI2_MISO: no longer U8.7 (DRDY)
- net SPI2_MOSI: no longer U8.4 (SDA/SDI/SDO)
- net SPI2_SCK: no longer U8.1 (SCL/SPC)
- new net MAG_I2C_SCL: U8.1 (SCL/SPC)
- new net MAG_I2C_SDA: U8.4 (SDA/SDI/SDO)
- no-connect marks 4 -> 5
Other:
- note added: "Capacitors used when changing reference plane"
- note added: "Stitching Capacitors"
- note added: "±49.152gauss 3-axis magnetometer"
- note removed: "±50gauss 3-axis magnetometer"
- moved on the sheet: C23, C24, C25, C28, C30, C31, C32, U8, U9
